File: eda/rc-car-remote-kicad/rc-car-remote.kicad_pcb (KiCad board)
At the start: 2 copper layers, 120 x 48 mm, 42 parts, among them J1 USB_C_Receptacle_USB2.0_14P, J2 AVR-ISP-10, J3 nRF24L01+ Headers, Q1 IRLML6244, SW1 SW_SPST, U1 TPS3840, U2 MCP73831-2-OT, U3 MIC5225-3.3YM5, U4 ATmega164A-A, j4 B09Y2R1GLV, j5 B09Y2R1GLV

Commit message: - Uploading rc car remote gerber files - Updated the 3d models for the rc car circuit. Changed them all to .step
Parts:
- added REF**: M2, MountingHole:MountingHole_2.2mm_M2_DIN965_Pad, F.Cu at (97.2, 87.2)
- added REF**: M2, MountingHole:MountingHole_2.2mm_M2_DIN965_Pad, F.Cu at (202.8, 87.2)
- added REF**: M2, MountingHole:MountingHole_2.2mm_M2_DIN965_Pad, F.Cu at (97.2, 120.8)
- added REF**: M2, MountingHole:MountingHole_2.2mm_M2_DIN965_Pad, F.Cu at (202.8, 120.8)
- moved D1 72.1 mm to (128.9, 86.7)
- moved R4 72.1 mm to (128.4, 82.2)
- moved J1 0.50 mm to (150.0, 82.5)
- renumbered 3.3V1 to 3.3V, CE1 to CE, CSN1 to CSN, Gnd1 to Gnd, LBtn1 to LBtn, LXaxis1 to LXaxis, MISO1 to MISO, MOSI1 to MOSI, RBtn1 to RBtn, RYaxis1 to RYaxis, SCK1 to SCK
Routing:
- net /U1-Reset: track 48.7 -> 50.7 mm, vias 1 -> 3
- net /LBtn: track 69.6 -> 70.8 mm
- net /RBtn: track 53.4 -> 54.7 mm
- net /5V USB: track 9.88 -> 8.82 mm
- net Net-(J1-CC2): track 4.42 -> 3.92 mm
- net Net-(J1-CC1): track 4.42 -> 3.92 mm
Other:
- board text added: "QB.Creates"
- board text added: "pcb-rc-car-remote-A1"
